Commit message: Attempted changes to control xacros

File: ros2/arm_robot_moveit_config/config/default_xacro/arm_robot_description.urdf.xacro (robot description, xacro)
@@ -2,12 +2,7 @@
 <robot xmlns:xacro="http://www.ros.org/wiki/xacro" name="arm_robot_description">
     <xacro:arg name="initial_positions_file" default="initial_positions.yaml" />
-    <xacro:arg name="use_nominal_extrinsics" default="false"/>
     <!-- Import arm_robot_description urdf file -->
     <xacro:include filename="$(find arm_robot_description)/urdf/arm_robot_description.urdf" />
-    <!-- Import depth camera -->
-    <xacro:include filename="$(find arm_robot_description)/urdf/_d405.urdf.xacro" />
-    <xacro:sensor_d405 parent="camera_link" use_nominal_extrinsics="$(arg use_nominal_extrinsics)">
-    <origin xyz="0 0 0.00129" rpy="0 -1.5707963268 -1.5707963268"/>
-    </xacro:sensor_d405>
+    <!-- Import control_xacro -->
     <xacro:include filename="arm_robot_description.ros2_control.xacro" />
     <xacro:arm_robot_description_ros2_control name="FakeSystem" initial_positions_file="$(arg initial_positions_file)"/>

File: ros2/arm_robot_moveit_config/config/dynamixel_xacro/arm_robot_description.ros2_control.xacro (robot description, xacro)
@@ -2,56 +2,51 @@
 <robot xmlns:xacro="http://www.ros.org/wiki/xacro">
     <xacro:macro name="arm_robot_description_ros2_control" params="name initial_positions_file">
-        <xacro:property name="initial_positions" value="${xacro.load_yaml(initial_positions_file)['initial_positions']}"/>
+    <xacro:property name="initial_positions" value="${xacro.load_yaml(initial_positions_file)['initial_positions']}"/>
         <ros2_control name="${name}" type="system">
             <hardware>
-                <!-- By default, set up controllers for simulation. This won't work on real hardware -->
-                <plugin>mock_components/GenericSystem</plugin>
+                <plugin>dynamixel_hardware/DynamixelHardware</plugin>
+        	<param name="usb_port">/dev/ttyUSB0</param>
+        	<param name="baud_rate">1000000</param>
             </hardware>
             <joint name="shoulder_joint">
+            	<param name="id">11</param>
                 <command_interface name="position"/>
                 <command_interface name="velocity"/>
                 <state_interface name="position">
-                  <param name="initial_value">${initial_positions['shoulder_joint']}</param>
-                </state_interface>
                 <state_interface name="velocity"/>
             </joint>
             <joint name="upperarm_joint">
+            	<param name="id">12</param>
                 <command_interface name="position"/>
                 <command_interface name="velocity"/>
                 <state_interface name="position">
-                  <param name="initial_value">${initial_positions['upperarm_joint']}</param>
-                </state_interface>
                 <state_interface name="velocity"/>
             </joint>
             <joint name="forearm_joint">
+            	<param name="id">13</param>
                 <command_interface name="position"/>
                 <command_interface name="velocity"/>
                 <state_interface name="position">
-                  <param name="initial_value">${initial_positions['forearm_joint']}</param>
-                </state_interface>
                 <state_interface name="velocity"/>
             </joint>
             <joint name="wrist_joint">
+            	<param name="id">14</param>
                 <command_interface name="position"/>
                 <command_interface name="velocity"/>
                 <state_interface name="position">
-                  <param name="initial_value">${initial_positions['wrist_joint']}</param>
-                </state_interface>
                 <state_interface name="velocity"/>
             </joint>
             <joint name="frame_joint">
+            	<param name="id">15</param>
                 <command_interface name="position"/>
                 <command_interface name="velocity"/>
                 <state_interface name="position">
-                  <param name="initial_value">${initial_positions['frame_joint']}</param>
-                </state_interface>
                 <state_interface name="velocity"/>
             </joint>
             <joint name="worm_joint">
+            	<param name="id">16</param>
                 <command_interface name="position"/>
                 <command_interface name="velocity"/>
                 <state_interface name="position">
-                  <param name="initial_value">${initial_positions['worm_joint']}</param>
-                </state_interface>
                 <state_interface name="velocity"/>
             </joint>

File: ros2/arm_robot_moveit_config/config/realsense_xacro/arm_robot_description.urdf.xacro (robot description, xacro)
@@ -10,5 +10,5 @@
     <origin xyz="0 0 0.00129" rpy="0 -1.5707963268 -1.5707963268"/>
     </xacro:sensor_d405>
-    <xacro:include filename="arm_robot_description.ros2_control.xacro" />
-    <xacro:arm_robot_description_ros2_control name="FakeSystem" initial_positions_file="$(arg initial_positions_file)"/>
+    <!--<xacro:include filename="arm_robot_description.ros2_control.xacro" />
+    <xacro:arm_robot_description_ros2_control name="FakeSystem" initial_positions_file="$(arg initial_positions_file)"/>-->
 </robot>
