Commit message: fixing ros2_control to use dynamixel
- modified arm_robot_description.urdf.xacro with a line from the OpenManipulator-X
- changed USB port (was USB0, now ACM0) and baud rate (was 1000000, now 115200) for DynamixelHardware in arm_robot_description.ros2_control.xacro
- created demo2.launch.py because the original demo.launch.py is harder to customize
- demo2.launch.py causes the ARM to rapidly move to a preset position (horizontal) excluding joint 1, but terminal output says missing/incorrect state and command interfaces

File: ros2/arm_robot_moveit_config/config/arm_robot_description.ros2_control.xacro (robot description, xacro)
@@ -2,56 +2,51 @@
 <robot xmlns:xacro="http://www.ros.org/wiki/xacro">
     <xacro:macro name="arm_robot_description_ros2_control" params="name initial_positions_file">
-        <xacro:property name="initial_positions" value="${xacro.load_yaml(initial_positions_file)['initial_positions']}"/>
+    <xacro:property name="initial_positions" value="${xacro.load_yaml(initial_positions_file)['initial_positions']}"/>
         <ros2_control name="${name}" type="system">
             <hardware>
-                <!-- By default, set up controllers for simulation. This won't work on real hardware -->
-                <plugin>mock_components/GenericSystem</plugin>
+                <plugin>dynamixel_hardware/DynamixelHardware</plugin>
+        	<param name="usb_port">/dev/ttyACM0</param>
+        	<param name="baud_rate">115200</param> <!-- or 1000000? -->
             </hardware>
             <joint name="shoulder_joint">
+            	<param name="id">1</param>
                 <command_interface name="position"/>
                 <command_interface name="velocity"/>
-                <state_interface name="position">
-                  <param name="initial_value">${initial_positions['shoulder_joint']}</param>
-                </state_interface>
+                <state_interface name="position"/>
                 <state_interface name="velocity"/>
             </joint>
             <joint name="upperarm_joint">
+            	<param name="id">2</param>
                 <command_interface name="position"/>
                 <command_interface name="velocity"/>
-                <state_interface name="position">
-                  <param name="initial_value">${initial_positions['upperarm_joint']}</param>
-                </state_interface>
+                <state_interface name="position"/>
                 <state_interface name="velocity"/>
             </joint>
             <joint name="forearm_joint">
+            	<param name="id">3</param>
                 <command_interface name="position"/>
                 <command_interface name="velocity"/>
-                <state_interface name="position">
-                  <param name="initial_value">${initial_positions['forearm_joint']}</param>
-                </state_interface>
+                <state_interface name="position"/>
                 <state_interface name="velocity"/>
             </joint>
             <joint name="wrist_joint">
+            	<param name="id">4</param>
                 <command_interface name="position"/>
                 <command_interface name="velocity"/>
-                <state_interface name="position">
-                  <param name="initial_value">${initial_positions['wrist_joint']}</param>
-                </state_interface>
+                <state_interface name="position"/>
                 <state_interface name="velocity"/>
             </joint>
             <joint name="frame_joint">
+            	<param name="id">5</param>
                 <command_interface name="position"/>
                 <command_interface name="velocity"/>
-                <state_interface name="position">
-                  <param name="initial_value">${initial_positions['frame_joint']}</param>
-                </state_interface>
+                <state_interface name="position"/>
                 <state_interface name="velocity"/>
             </joint>
             <joint name="worm_joint">
+            	<param name="id">6</param>
                 <command_interface name="position"/>
                 <command_interface name="velocity"/>
-                <state_interface name="position">
-                  <param name="initial_value">${initial_positions['worm_joint']}</param>
-                </state_interface>
+                <state_interface name="position"/>
                 <state_interface name="velocity"/>
             </joint>

File: ros2/arm_robot_moveit_config/config/dynamixel_xacro/arm_robot_description.ros2_control.xacro (robot description, xacro)
@@ -6,47 +6,47 @@
             <hardware>
                 <plugin>dynamixel_hardware/DynamixelHardware</plugin>
-        	<param name="usb_port">/dev/ttyUSB0</param>
+        	<param name="usb_port">/dev/ttyACM0</param>
         	<param name="baud_rate">1000000</param>
             </hardware>
             <joint name="shoulder_joint">
-            	<param name="id">11</param>
+            	<param name="id">1</param>
                 <command_interface name="position"/>
                 <command_interface name="velocity"/>
-                <state_interface name="position">
+                <state_interface name="position"/>
                 <state_interface name="velocity"/>
             </joint>
             <joint name="upperarm_joint">
-            	<param name="id">12</param>
+            	<param name="id">2</param>
                 <command_interface name="position"/>
                 <command_interface name="velocity"/>
-                <state_interface name="position">
+                <state_interface name="position"/>
                 <state_interface name="velocity"/>
             </joint>
             <joint name="forearm_joint">
-            	<param name="id">13</param>
+            	<param name="id">3</param>
                 <command_interface name="position"/>
                 <command_interface name="velocity"/>
-                <state_interface name="position">
+                <state_interface name="position"/>
                 <state_interface name="velocity"/>
             </joint>
             <joint name="wrist_joint">
-            	<param name="id">14</param>
+            	<param name="id">4</param>
                 <command_interface name="position"/>
                 <command_interface name="velocity"/>
-                <state_interface name="position">
+                <state_interface name="position"/>
                 <state_interface name="velocity"/>
             </joint>
             <joint name="frame_joint">
-            	<param name="id">15</param>
+            	<param name="id">5</param>
                 <command_interface name="position"/>
                 <command_interface name="velocity"/>
-                <state_interface name="position">
+                <state_interface name="position"/>
                 <state_interface name="velocity"/>
             </joint>
             <joint name="worm_joint">
-            	<param name="id">16</param>
+            	<param name="id">6</param>
                 <command_interface name="position"/>
                 <command_interface name="velocity"/>
-                <state_interface name="position">
+                <state_interface name="position"/>
                 <state_interface name="velocity"/>
             </joint>
