Commit message: Updated SRDF according to new limits and adjusted preference things in other files

File: ros2/arm_robot_description/urdf/test_d405_camera.urdf.xacro (robot description, xacro)
@@ -6,4 +6,5 @@
   <xacro:sensor_d405 parent="camera_link" use_nominal_extrinsics="$(arg use_nominal_extrinsics)">
     <origin xyz="0 0 0" rpy="0 0 0"/>
+    <!-- <origin xyz="0 0 0.00129" rpy="0 -1.5707963268 -1.5707963268"/> --> <!-- consider using this one to reposition and orient pointcloud correctly?-->
   </xacro:sensor_d405>
 </robot>
