Commit message: Added pointcloud, fixed(?) wrist behavior in opencm_command3

File: ros2/arm_robot_description/urdf/_d405.urdf.xacro (robot description, xacro)
@@ -23,5 +23,5 @@
   <xacro:include filename="$(find arm_robot_description)/urdf/_materials.urdf.xacro" />
   <xacro:include filename="$(find arm_robot_description)/urdf/_usb_plug.urdf.xacro" />
-  <xacro:macro name="sensor_d405" params="parent *origin name:=camera2 use_nominal_extrinsics:=false">
+  <xacro:macro name="sensor_d405" params="parent *origin name:=depcamera use_nominal_extrinsics:=false">
     <xacro:arg name="add_plug" default="false" />
     <xacro:property name="M_PI" value="3.1415926535897931" />

File: ros2/arm_robot_description/urdf/arm_robot_description.urdf (robot description, URDF)
Before this commit: robot arm_robot_description, 14 links, 13 joints
Joints:
- joint camera_joint: origin xyz=0.028329 0.016933 0.06075 rpy=0 0 -1.0472 -> xyz=0.028329 0.016933 0.06075 rpy=-1.5707963268 -1.5707963268 -1.0472

File: ros2/arm_robot_moveit_config/config/arm_robot_description.urdf.xacro (robot description, xacro)
@@ -8,5 +8,5 @@
     <xacro:include filename="$(find arm_robot_description)/urdf/_d405.urdf.xacro" />
     <xacro:sensor_d405 parent="camera_link" use_nominal_extrinsics="$(arg use_nominal_extrinsics)">
-    <origin xyz="0 0 0.00129" rpy="0 -1.5707963268 -1.5707963268"/>
+    <origin xyz="0.00129 0 0" rpy="0 0 0"/> <!-- this only applies to model of camera, not the pointcloud -->
     </xacro:sensor_d405>
     <!-- Import control_xacro -->
