Commit message: Include depth camera config

File: ros2/arm_robot_description/urdf/arm_robot_description.urdf (robot description, URDF)
Before this commit: robot arm_robot_description, 14 links, 13 joints
Links:
- link base_link: mass 0.163939534292526 -> None
- link camera_link: geometry 

Commit message: Removed dynamixel control stuff so that opencm_command3 works

File: ros2/arm_robot_description/urdf/arm_robot_description.urdf (robot description, URDF)
Before this commit: robot arm_robot_description, 14 links, 13 joints
Joints:
- joint forearm_joint: limit lower=-1.95 upper=1.95 effort=0 velocity=0 -> lower=-1.5708 upper=1.5708 effort=0 velocity=0
- joint upperarm_joint: limit lower=-2.24 upper=2.24 effort=0 velocity=0 -> lower=-1.5708 upper=1.5708 effort=0 velocity=0

File: ros2/arm_robot_moveit_config/config/arm_robot_description.ros2_control.xacro (robot description, xacro)
@@ -2,52 +2,56 @@
 <robot xmlns:xacro="http://www.ros.org/wiki/xacro">
     <xacro:macro name="arm_robot_description_ros2_control" params="name initial_positions_file">
-    <xacro:property name="initial_positions" value="${xacro.load_yaml(initial_positions_file)['initial_positions']}"/>
+        <xacro:property name="initial_positions" value="${xacro.load_yaml(initial_positions_file)['initial_positions']}"/>
         <ros2_control name="${name}" type="system">
             <hardware>
-                <plugin>dynamixel_hardware/DynamixelHardware</plugin>
-        	<param name="usb_port">/dev/ttyACM0</param>
-        	<param name="baud_rate">115200</param> <!-- or 1000000? -->
-        	<param name="use_dummy">true</param>
+                <!-- By default, set up controllers for simulation. This won't work on real hardware -->
+                <plugin>mock_components/GenericSystem</plugin>
             </hardware>
             <joint name="shoulder_joint">
-            	<param name="id">1</param>
                 <command_interface name="position"/>
                 <command_interface name="velocity"/>
-                <state_interface name="position"/>
+                <state_interface name="position">
+                  <param name="initial_value">${initial_positions['shoulder_joint']}</param>
+                </state_interface>
                 <state_interface name="velocity"/>
             </joint>
             <joint name="upperarm_joint">
-            	<param name="id">2</param>
                 <command_interface name="position"/>
                 <command_interface name="velocity"/>
-                <state_interface name="position"/>
+                <state_interface name="position">
+                  <param name="initial_value">${initial_positions['upperarm_joint']}</param>
+                </state_interface>
                 <state_interface name="velocity"/>
             </joint>
             <joint name="forearm_joint">
-            	<param name="id">3</param>
                 <command_interface name="position"/>
                 <command_interface name="velocity"/>
-                <state_interface name="position"/>
+                <state_interface name="position">
+                  <param name="initial_value">${initial_positions['forearm_joint']}</param>
+                </state_interface>
                 <state_interface name="velocity"/>
             </joint>
             <joint name="wrist_joint">
-            	<param name="id">4</param>
                 <command_interface name="position"/>
                 <command_interface name="velocity"/>
-                <state_interface name="position"/>
+                <state_interface name="position">
+                  <param name="initial_value">${initial_positions['wrist_joint']}</param>
+                </state_interface>
                 <state_interface name="velocity"/>
             </joint>
             <joint name="frame_joint">
-            	<param name="id">5</param>
                 <command_interface name="position"/>
                 <command_interface name="velocity"/>
-                <state_interface name="position"/>
+                <state_interface name="position">
+                  <param name="initial_value">${initial_positions['frame_joint']}</param>
+                </state_interface>
                 <state_interface name="velocity"/>
             </joint>
             <joint name="worm_joint">
-            	<param name="id">6</param>
                 <command_interface name="position"/>
                 <command_interface name="velocity"/>
-                <state_interface name="position"/>
+                <state_interface name="position">
+                  <param name="initial_value">${initial_positions['worm_joint']}</param>
+                </state_interface>
                 <state_interface name="velocity"/>
             </joint>

File: ros2/arm_robot_moveit_config/config/arm_robot_description.urdf.xacro (robot description, xacro)
@@ -10,6 +10,6 @@
     <origin xyz="0 0 0.00129" rpy="0 -1.5707963268 -1.5707963268"/>
     </xacro:sensor_d405>
+    <!-- Import control_xacro -->
     <xacro:include filename="arm_robot_description.ros2_control.xacro" />
-    <!--<xacro:arm_robot_description_ros2_control name="FakeSystem" initial_positions_file="$(arg initial_positions_file)"/>--> <!-- original -->
-    <xacro:arm_robot_description_ros2_control name="arm_robot_description_ros2_control" initial_positions_file="$(arg initial_positions_file)"/> <!-- imitated from open_manipulator_x.urdf.xacro -->
+    <xacro:arm_robot_description_ros2_control name="FakeSystem" initial_positions_file="$(arg initial_positions_file)"/>
 </robot>

Commit message: Created vision_motion.py, expanded one joint limit

File: ros2/arm_robot_description/urdf/arm_robot_description.urdf (robot description, URDF)
Before this commit: robot arm_robot_description, 14 links, 13 joints
Joints:
- joint forearm_joint: limit lower=-1.5708 upper=1.5708 effort=0 velocity=0 -> lower=-1.570796327 upper=1.570796327 effort=0 velocity=0; origin xyz=0.035651 -0.14 0 rpy=3.1416 0 3.1416 -> xyz=0.035651 -0.14 0 rpy=3.1415926536 0 3.1415926536
- joint frame_joint: limit lower=-3.1415 upper=3.1415 effort=0 velocity=0 -> lower=-3.1415926536 upper=3.1415926536 effort=0 velocity=0
- joint left_inner_joint: origin xyz=0.02616 -0.025311 0.035 rpy=3.1416 0.37217 2.0944 -> xyz=0.02616 -0.025311 0.035 rpy=3.1415926536 0.37217 2.0944
- joint left_outer_joint: origin xyz=0.03116 -0.033971 0.035 rpy=3.1416 0.37217 2.0944 -> xyz=0.03116 -0.033971 0.035 rpy=3.1415926536 0.37217 2.0944
- joint right_inner_joint: origin xyz=-0.00017949 0.040311 0.035 rpy=3.1416 0.37217 -1.0472 -> xyz=-0.00017949 0.040311 0.035 rpy=3.1415926536 0.37217 -1.0472
- joint right_outer_joint: origin xyz=-0.0095096 0.046471 0.035 rpy=3.1416 0.37217 -1.0472 -> xyz=-0.0095096 0.046471 0.035 rpy=3.1415926536 0.37217 -1.0472
- joint shoulder_joint: limit lower=-3.1415 upper=3.1415 effort=0 velocity=0 -> lower=-3.1415926536 upper=3.1415926536 effort=0 velocity=0; origin xyz=0.042 -0.042 0.052082 rpy=1.5708 0 -3.1416 -> xyz=0.042 -0.042 0.052082 rpy=1.570796327 0 -3.1415926536
- joint upperarm_joint: limit lower=-1.5708 upper=1.5708 effort=0 velocity=0 -> lower=-1.570796327 upper=1.832596 effort=0 velocity=0; origin xyz=-0.036613 0.084019 0 rpy=3.1416 0 0 -> xyz=-0.036613 0.084019 0 rpy=3.1415926536 0 0
- joint worm_joint: limit lower=0 upper=3.1415 effort=0 velocity=0 -> lower=0 upper=3.1415926536 effort=0 velocity=0; origin xyz=0.01299 0.0075 0.038 rpy=3.1416 0 -3.0183 -> xyz=0.01299 0.0075 0.038 rpy=3.1415926536 0 -3.0183
- joint wrist_joint: origin xyz=-0.035049 -0.145 0 rpy=0 -0.96942 -1.5708 -> xyz=-0.035049 -0.145 0 rpy=0 -0.96942 -1.570796327

Commit message: Adjustments for RViz

File: ros2/arm_robot_description/urdf/arm_robot_description.urdf (robot description, URDF)
Before this commit: robot arm_robot_description, 14 links, 13 joints
Joints:
- joint upperarm_joint: limit lower=-1.570796327 upper=1.832596 effort=0 velocity=0 -> lower=-1.570796327 upper=1.570796327 effort=0 velocity=0
